Commit message: Housing my robot insider room and Package
Integrating my robot inside my house.

File: catkin_wsP2/src/my_robot/urdf/my_robot.xacro (robot description, xacro)
@@ -105,5 +105,5 @@
       <origin xyz="0 0 0" rpy="0 1.5707 1.5707"/>
       <geometry>
-        <cylinder length="0.0499" radius="0.099" />
+        <cylinder length="0.05" radius="0.1" />
       </geometry>
     </collision>
@@ -124,5 +124,5 @@
       <origin xyz="0 0 0" rpy="0 1.5707 1.5707"/>
       <geometry>
-        <cylinder length="0.0499" radius="0.099" />
+        <cylinder length="0.05" radius="0.1" />
       </geometry>
     </collision>
